Commit message: mocap: 固化 frame0 跟踪与仿真位姿诊断
确认当前 wrist 跟踪和 approaching 到 frame0 流程正常。

加入 frame0 21 点/20 骨段 MuJoCo 对照骨架，并保留已知问题：H5 frame0 数据映射到 sim 后的位姿不正确。

File: src/pico_body_tianji/assets/marvin_m6_ccs/urdf/marvin_m6_s_ccs_696_v4_wuji2.urdf (robot description, URDF)
Before this commit: robot Marvin M6-S-CCS-696-V4.0_Base_and_Stand_Asm urdf, 48 links, 47 joints
Links:
- added link marker_mocap, mass 0.0167124616872421; visual cylinder length=0.07 radius=0.004; visual cylinder length=0.07 radius=0.004
- added link marker_tianji
- added link marker_wuji2
- link r_mount_frame: geometry visual sphere radius=0.004
- link r_wrist: geometry visual cylinder length=0.09 radius=0.005; visual cylinder length=0.09 radius=0.005
Joints:
- added joint JointMarker_R: type fixed, parent TCP_Link_R, child marker_tianji, origin xyz=0 0 0 rpy=-1.5707963267948966 -1.5707963267948966 0
- added joint marker_tianji_to_mocap: type fixed, parent marker_tianji, child marker_mocap, origin xyz=0.004 0 0 rpy=0 0 0
- added joint marker_wuji2: type fixed, parent marker_mocap, child marker_wuji2, origin xyz=0.004 0 0 rpy=0 0 0
- joint JointWuji2_R: origin xyz=0 0 0 rpy=3.14159265359 0 1.57079632679 -> xyz=0 0 0 rpy=3.141592653589793 -1.5707963267948966 0; parent TCP_Link_R -> marker_wuji2
- joint r_mount_frame_to_base: origin xyz=0.003 0.00025 -0.0285 rpy=3.141592653589793 0 0 -> xyz=0.003 -0.00025 0.0285 rpy=0 0 0

File: src/pico_body_tianji/assets/wuji2_right/right_with_mount_marker.urdf (robot description, URDF)
Before this commit: robot wujihand-right, 28 links, 27 joints
Links:
- link r_index_finger_distal: geometry collision mesh filename=collision/r_index_finger_distal_convex_0.obj; visual mesh filename=package://pico_body_tianji/assets/marvin_m6_ccs/meshes/wuji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
- link r_index_finger_middle: geometry collision mesh filename=collision/r_index_finger_middle_convex_0.obj; visual mesh filename=package://pico_body_tianji/assets/marvin_m6_ccs/meshes/wuji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
- link r_index_finger_proximal: geometry collision mesh filename=collision/r_index_finger_proximal_convex_0.obj; collision mesh filename=collision/r_index_finger_proximal_convex_1.obj
- link r_index_finger_proximal_abd: geometry collision mesh filename=collision/r_index_finger_proximal_abd_convex_0.obj; visual mesh filename=package://pico_body_tianji/assets/marvin_m6_ccs/meshes/wuji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
- link r_index_finger_tip: geometry collision mesh filename=collision/r_index_finger_tip_convex_0.obj; visual mesh filename=package://pico_body_tianji/assets/marvin_m6_ccs/meshes/wuji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
- link r_middle_finger_distal: geometry collision mesh filename=collision/r_middle_finger_distal_convex_0.obj; visual mesh filename=package://pico_body_tianji/assets/marvin_m6_ccs/meshes/wuji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
- link r_middle_finger_middle: geometry collision mesh filename=collision/r_middle_finger_middle_convex_0.obj; visual mesh filename=package://pico_body_tianji/assets/marvin_m6_ccs/meshes/wuji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
- link r_middle_finger_proximal: geometry collision mesh filename=collision/r_middle_finger_proximal_convex_0.obj; collision mesh filename=collision/r_middle_finger_proximal_convex_1.obj
- link r_middle_finger_proximal_abd: geometry collision mesh filename=collision/r_middle_finger_proximal_abd_convex_0.obj; visual mesh filename=package://pico_body_tianji/assets/marvin_m6_ccs/meshes/wuji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
- link r_middle_finger_tip: geometry collision mesh filename=collision/r_middle_finger_tip_convex_0.obj; visual mesh filename=package://pico_body_tianji/assets/marvin_m6_ccs/meshes/wuji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
- link r_pinky_distal: geometry collision mesh filename=collision/r_pinky_distal_convex_0.obj; visual mesh filename=package://pico_body_tianji/assets/marvin_m6_ccs/meshes/wuji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
- link r_pinky_middle: geometry collision mesh filename=collision/r_pinky_middle_convex_0.obj; visual mesh filename=package://pico_body_tianji/assets/marvin_m6_ccs/meshes/wuji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
- link r_pinky_proximal: geometry collision mesh filename=collision/r_pinky_proximal_convex_0.obj; collision mesh filename=collision/r_pinky_proximal_convex_1.obj
- link r_pinky_proximal_abd: geometry collision mesh filename=collision/r_pinky_proximal_abd_convex_0.obj; visual mesh filename=package://pico_body_tianji/assets/marvin_m6_ccs/meshes/wuji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
- link r_pinky_tip: geometry collision mesh filename=collision/r_pinky_tip_convex_0.obj; visual mesh filename=package://pico_body_tianji/assets/marvin_m6_ccs/meshes/wuji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
- link r_ring_finger_distal: geometry collision mesh filename=collision/r_ring_finger_distal_convex_0.obj; visual mesh filename=package://pico_body_tianji/assets/marvin_m6_ccs/meshes/wuji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
- link r_ring_finger_middle: geometry collision mesh filename=collision/r_ring_finger_middle_convex_0.obj; visual mesh filename=package://pico_body_tianji/assets/marvin_m6_ccs/meshes/wuji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
- link r_ring_finger_proximal: geometry collision mesh filename=collision/r_ring_finger_proximal_convex_0.obj; collision mesh filename=collision/r_ring_finger_proximal_convex_1.obj
- link r_ring_finger_proximal_abd: geometry collision mesh filename=collision/r_ring_finger_proximal_abd_convex_0.obj; visual mesh filename=package://pico_body_tianji/assets/marvin_m6_ccs/meshes/wuji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
- link r_ring_finger_tip: geometry collision mesh filename=collision/r_ring_finger_tip_convex_0.obj; visual mesh filename=package://pico_body_tianji/assets/marvin_m6_ccs/meshes/wuji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
- link r_thumb_distal: geometry collision mesh filename=collision/r_thumb_distal_convex_0.obj; visual mesh filename=package://pico_body_tianji/assets/marvin_m6_ccs/meshes/wuji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
- link r_thumb_middle: geometry collision mesh filename=collision/r_thumb_middle_convex_0.obj; visual mesh filename=package://pico_body_tianji/assets/marvin_m6_ccs/meshes/wuji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
- link r_thumb_proximal: geometry collision mesh filename=collision/r_thumb_proximal_convex_0.obj; collision mesh filename=collision/r_thumb_proximal_convex_1.obj
- link r_thumb_proximal_abd: geometry collision mesh filename=collision/r_thumb_proximal_abd_convex_0.obj; visual mesh filename=package://pico_body_tianji/assets/marvin_m6_ccs/meshes/wuji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
- link r_thumb_tip: geometry collision mesh filename=collision/r_thumb_tip_convex_0.obj; visual mesh filename=package://pico_body_tianji/assets/marvin_m6_ccs/meshes/wuji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
- link r_wrist: geometry collision mesh filename=collision/r_wrist_convex_0.obj; visual mesh filename=package://pico_body_tianji/assets/marvin_m6_ccs/meshes/wuji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
Joints:
- joint r_base_to_mount: origin xyz=-0.003 0.00025 -0.0285 rpy=3.141592653589793 0 0 -> xyz=-0.003 0.00025 -0.0285 rpy=0 0 0

Commit message: mocap: r_base 端点与坐标轴对齐
回放端点为 wuji2 r_base（URDF link）；r_base 轴随 URDF FK 运动，Manus 骨架轴与 r_base 轴均用 RGB 显示并隐藏 URDF 自带轴。

Manus→r_base 外参绕 base z +90° 补偿数据朝向；45 项回放/readiness 测试通过。

File: src/pico_body_tianji/assets/marvin_m6_ccs/urdf/marvin_m6_s_ccs_696_v4_wuji2.urdf (robot description, URDF)
Before this commit: robot Marvin M6-S-CCS-696-V4.0_Base_and_Stand_Asm urdf, 51 links, 50 joints
Links:
- link r_base: geometry visual cylinder length=0.09 radius=0.005; visual cylinder length=0.09 radius=0.005

Commit message: feat: 迁移动捕链路到 wuji2 beta1 右手并统一 z-up 世界坐标
- 接入最新版 hand2_beta1 右手 URDF 与 22 个实际引用 STL
- 组合链改为 TCP -> marker -> r_mount -> r_wrist -> fingers，移除虚构 r_base/Rx(pi)
- r_mount 作为 tianji_wrist 刚体定位的安装基准；Manus wrist 直接映射 r_wrist
- 为 r_mount 增加 FK 坐标轴可视化，随手臂末端移动
- 动捕/keyboard/live 按键映射由 y-up 改为 x-forward z-up 右手系
- 刚体默认名 right_arm/left_wrist 改为 tianji_wrist/left_back
- host_readiness/status 契约同步为 wuji2_r_wrist；文档与测试更新

File: src/pico_body_tianji/assets/marvin_m6_ccs/urdf/marvin_m6_s_ccs_696_v4_wuji2.urdf (robot description, URDF)
Before this commit: robot Marvin M6-S-CCS-696-V4.0_Base_and_Stand_Asm urdf, 51 links, 50 joints
Links:
- removed link r_base
- removed link r_mount_frame
- added link r_mount, mass 0.069; visual cylinder length=0.06 radius=0.004; visual cylinder length=0.06 radius=0.004
- link r_index_finger_distal: mass 0.014 -> 0.0078
- link r_index_finger_middle: mass 0.0165 -> 0.0212
- link r_index_finger_proximal: mass 0.0032 -> 0.0116
- link r_index_finger_proximal_abd: mass 0.033 -> 0.0339
- link r_index_finger_tip: mass 0.00318 -> None; geometry 
- link r_middle_finger_distal: mass 0.014 -> 0.0078
- link r_middle_finger_middle: mass 0.0165 -> 0.0212
- link r_middle_finger_proximal: mass 0.0032 -> 0.0116
- link r_middle_finger_proximal_abd: mass 0.033 -> 0.0339
- link r_middle_finger_tip: mass 0.00318 -> None; geometry 
- link r_pinky_distal: mass 0.014 -> 0.0078
- link r_pinky_middle: mass 0.0165 -> 0.0188
- link r_pinky_proximal: mass 0.0032 -> 0.0116
- link r_pinky_proximal_abd: mass 0.033 -> 0.0304
- link r_pinky_tip: mass 0.00318 -> None; geometry 
- link r_ring_finger_distal: mass 0.014 -> 0.0078
- link r_ring_finger_middle: mass 0.0165 -> 0.0212
- link r_ring_finger_proximal: mass 0.0032 -> 0.0116
- link r_ring_finger_proximal_abd: mass 0.033 -> 0.0339
- link r_ring_finger_tip: mass 0.00318 -> None; geometry 
- link r_thumb_distal: mass 0.0165 -> 0.0159
- link r_thumb_middle: mass 0.0165 -> 0.0358
- link r_thumb_proximal: mass 0.0075 -> 0.011
- link r_thumb_proximal_abd: mass 0.0248 -> 0.0336
- link r_thumb_tip: mass 0.0041 -> None; geometry 
- link r_wrist: mass 0.16914 -> 0.2323
Joints:
- removed joint r_base_to_wrist
- removed joint r_mount_frame_to_base
- added joint r_wrist_fixed: type fixed, parent r_mount, child r_wrist, origin xyz=0.003 0.00025016 -0.0285 rpy=0 0 1.6399E-05
- joint JointWuji2_R: child r_mount_frame -> r_mount; origin xyz=0 0 0 rpy=3.141592653589793 -1.5707963267948966 0 -> xyz=0 0 0 rpy=0 -1.5707963267948966 0
- joint r_index_finger_dip: limit lower=-1.047 upper=1.57 effort=0.3 velocity=13.5 -> lower=-1.0470 upper=1.5700 effort=0.3000 velocity=13.5; origin xyz=0 0 -0.0295000000000005 rpy=0 0 0 -> xyz=0 0 -0.0295 rpy=0 0 0
- joint r_index_finger_mcp_abd: limit lower=-0.698 upper=0.698 effort=0.2 velocity=8.11 -> lower=-0.6980 upper=0.6980 effort=0.2000 velocity=8.11; origin xyz=0 -0.0015851418713986 -0.0144630452761802 rpy=-0.0265261580297666 0 0 -> xyz=0 -0.001201 -0.0145 rpy=0 0 0
- joint r_index_finger_mcp_flex: limit lower=-1.047 upper=1.57 effort=2.0 velocity=8.203 -> lower=-1.0470 upper=1.5700 effort=2.0000 velocity=8.203; origin xyz=0.0203528654190901 -0.00336011581054318 -0.070679437897893 rpy=-0.01045839529445 -0.104348822398209 0.100075675935804 -> xyz=0.0226609454742 -0.00332513161729 -0.069975 rpy=-0.039792 -0.13705 0.100403601
- joint r_index_finger_pip: limit lower=-1.047 upper=2.094 effort=0.3 velocity=12.86 -> lower=-1.0470 upper=2.0940 effort=0.3000 velocity=12.86; origin xyz=0 0 -0.0376000000000001 rpy=0 0 0 -> xyz=0 0 -0.0376 rpy=0 0 0
- joint r_index_finger_tip_fixed: origin xyz=0 -0.00167219746761747 -0.025 rpy=0 0 0 -> xyz=0 0 -0.02475 rpy=0 0 0
- joint r_middle_finger_dip: limit lower=-1.047 upper=1.57 effort=0.3 velocity=13.5 -> lower=-1.0470 upper=1.5700 effort=0.3000 velocity=13.5; origin xyz=0 0 -0.0295000000000004 rpy=0.0344012194700258 0 0 -> xyz=0 0 -0.0295 rpy=0 0 0
- joint r_middle_finger_mcp_abd: limit lower=-0.698 upper=0.698 effort=0.2 velocity=8.11 -> lower=-0.6980 upper=0.6980 effort=0.2000 velocity=8.11; origin xyz=0 -0.00120098018725689 -0.0145000000001074 rpy=0 0 0 -> xyz=0 -0.001201 -0.0145 rpy=0 0 0
- joint r_middle_finger_mcp_flex: limit lower=-1.047 upper=1.57 effort=2.0 velocity=8.203 -> lower=-1.0470 upper=1.5700 effort=2.0000 velocity=8.203; origin xyz=-0.00147348225616674 -0.00833993676457262 -0.0739026139528614 rpy=-0.0344328490772506 0.0438522369960471 -0.000721508035749565 -> xyz=0.000952063839631 -0.00830297561401 -0.07392 rpy=-0.03391 0.011037 -0.000715349
- joint r_middle_finger_pip: limit lower=-1.047 upper=2.094 effort=0.3 velocity=12.86 -> lower=-1.0470 upper=2.0940 effort=0.3000 velocity=12.86; origin xyz=0 0 -0.0376000000000002 rpy=0 0 0 -> xyz=0 0 -0.0376 rpy=0 0 0
- joint r_middle_finger_tip_fixed: origin xyz=0 -0.00253106895306443 -0.0249276941237159 rpy=-0.0344012194700258 0 0 -> xyz=0 0 -0.02475 rpy=0 0 0
- joint r_pinky_dip: limit lower=-1.047 upper=1.57 effort=0.3 velocity=13.5 -> lower=-1.0470 upper=1.5700 effort=0.3000 velocity=13.5
- joint r_pinky_mcp_abd: limit lower=-0.698 upper=0.698 effort=0.2 velocity=8.11 -> lower=-0.6980 upper=0.6980 effort=0.2000 velocity=8.11
- joint r_pinky_mcp_flex: limit lower=-1.047 upper=1.57 effort=2.0 velocity=8.203 -> lower=-1.0470 upper=1.5700 effort=2.0000 velocity=8.203; origin xyz=-0.039145 -0.00076138 -0.054041 rpy=-0.035083 0.2813 -0.13736 -> xyz=-0.0373510120379 -0.000733757480852 -0.055296 rpy=-0.029938 0.24886 -0.136016399
- joint r_pinky_pip: limit lower=-1.047 upper=2.094 effort=0.3 velocity=12.86 -> lower=-1.0470 upper=2.0940 effort=0.3000 velocity=12.86
- joint r_pinky_tip_fixed: origin xyz=0 -0.00167219746761752 -0.025 rpy=0 0 0 -> xyz=0 0 -0.02475 rpy=0 0 0
- joint r_ring_finger_dip: limit lower=-1.047 upper=1.57 effort=0.3 velocity=13.5 -> lower=-1.0470 upper=1.5700 effort=0.3000 velocity=13.5; origin xyz=0 0 -0.0295000000000005 rpy=0 0 0 -> xyz=0 0 -0.0295 rpy=0 0 0
- joint r_ring_finger_mcp_abd: limit lower=-0.698 upper=0.698 effort=0.2 velocity=8.11 -> lower=-0.6980 upper=0.6980 effort=0.2000 velocity=8.11; origin xyz=0 -0.00120098018725689 -0.0145000000001074 rpy=0 0 0 -> xyz=0 -0.001201 -0.0145 rpy=0 0 0
- joint r_ring_finger_mcp_flex: limit lower=-1.047 upper=1.57 effort=2.0 velocity=8.203 -> lower=-1.0470 upper=1.5700 effort=2.0000 velocity=8.203; origin xyz=-0.021878890103642 -0.0056255988899957 -0.0647140852094928 rpy=-0.0194350140122241 0.17433767952625 -0.0687489294023846 -> xyz=-0.0197440917212 -0.00559293621739 -0.0654 rpy=-0.016655 0.14163 -0.068319399
- joint r_ring_finger_pip: limit lower=-1.047 upper=2.094 effort=0.3 velocity=12.86 -> lower=-1.0470 upper=2.0940 effort=0.3000 velocity=12.86; origin xyz=0 0 -0.0376000000000001 rpy=0 0 0 -> xyz=0 0 -0.0376 rpy=0 0 0
- joint r_ring_finger_tip_fixed: origin xyz=0 -0.00167219746761748 -0.025 rpy=0 0 0 -> xyz=0 0 -0.02475 rpy=0 0 0
- joint r_thumb_cmc_abd: limit lower=-1.484 upper=0.698 effort=0.6 velocity=11.1 -> lower=-1.4840 upper=0.6980 effort=0.6000 velocity=11.1; origin xyz=0.000247879062961599 -0.000536579546410674 -0.0147535404706145 rpy=0.205291970332105 0.70050871717831 0.0252378802492596 -> xyz=0.00024788 -0.00053658 -0.014754 rpy=0.20529 0.70051 0.025238
- joint r_thumb_cmc_flex: limit lower=-1.187 upper=1.291 effort=0.6 velocity=8.587 -> lower=-1.1870 upper=1.2910 effort=0.6000 velocity=8.587; origin xyz=0.0166602520939135 0.00812974518139747 -0.0170173790088068 rpy=-1.59876884374798 -1.07116653994079 1.93704700103865 -> xyz=0.0172101334567 0.00813795777212 -0.016457 rpy=-1.6617 -1.059 1.992083601
- joint r_thumb_ip: limit lower=-1.047 upper=1.57 effort=0.3 velocity=13.5 -> lower=-1.0470 upper=1.5700 effort=0.3000 velocity=13.5; origin xyz=-4.99999999923513E-05 0.00385197213324594 -0.0347873872356727 rpy=0.110279740852306 0 0 -> xyz=-5E-05 0 -0.035 rpy=0 0 0
- joint r_thumb_mcp: limit lower=-1.047 upper=1.57 effort=0.3 velocity=12.86 -> lower=-1.0470 upper=1.5700 effort=0.3000 velocity=12.86; origin xyz=0 0 -0.032500002798739 rpy=-0.11027974085231 0.0872664625995901 0.567232006897994 -> xyz=0 0 -0.0325 rpy=0 0.087266 0.56723
- joint r_thumb_tip_fixed: origin xyz=0 -0.000557448922432543 -0.0276972900827579 rpy=0 0 0 -> xyz=0 0 -0.02978 rpy=0 0 0
